File: pcb/esphome-rgbcct-led-controller-esp32.kicad_sch (KiCad schematic)
At the start: 18 parts, among them J4 USB-C, U7 ESP32-C3-MINI-1, U9 74AHCT32

Commit message: Add Energy sensor with Wh units
Co-authored-by: Copilot <copilot@github.com>
Parts:
- J2, SW1, SW2: value ~ -> (none)
