File: pcb/esphome-rgbcct-led-controller.kicad_sch (KiCad schematic)
At the start: 2 parts

Commit message: Add Energy sensor with Wh units
Co-authored-by: Copilot <copilot@github.com>
Parts:
- MH1, MH2: value ~ -> (none)
