File: pcb-expansion-rev-a/esphome-rgbcct-led-controller-expansion.kicad_sch (KiCad schematic)
At the start: 19 parts, among them J2 Conn_01x04, J3 Conn_01x02, J4 Conn_01x02, J5 Conn_01x02, J6 Conn_01x02, U1 ADS1015, U2 REF35300QDBVR

Commit message: Update Expansion Rev A Schematic Add more details for connecting sensors
Other:
- note added: "Amazon and AliExpress"
- note added: "I^{2}C Temp Sensor Connections"
- moved on the sheet: C1, C2, C3, C4, C5, J1, J2, J3, J4, J5, J6, MH1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

Commit message: Finish updating to Kicad 10
Parts:
- J1, MH1, MH2: value ~ -> (none)
