File: pcb-expansion-rev-b/esphome-rgbcct-led-controller-expansion.kicad_sch (KiCad schematic)
At the start: 19 parts, among them J2 Conn_01x04, J3 Conn_01x02, J4 Conn_01x02, J5 Conn_01x02, J6 Conn_01x02, U1 ADS1015, U2 REF35300QDBVR

Commit message: Finish updating to Kicad 10
Parts:
- J1, MH1, MH2: value ~ -> (none)
